Commit message: Add Dockerfile and ROS2 workspace

File: install/dd_robot/share/dd_robot/urdf/common_properties.xacro (robot description, xacro)
@@ -1,40 +1 @@
-<?xml version="1.0"?>
-<robot name="dd_robot" xmlns:xacro="http://www.ros.org/wiki/xacro">
-    <material name="green">
-        <color rgba="0 0.6 0 1" />
-    </material>
-    <material name="gray">
-        <color rgba="0.7 0.7 0.7 1" />
-    </material>
-    <xacro:macro name="box_inertia" params="m x y z o_xyz o_rpy">
-        <xacro:property name="ixx" value="${(m/12.0)*(y**2 + z**2)}"/>
-        <xacro:property name="iyy" value="${(m/12.0)*(x**2 + z**2)}"/>
-        <xacro:property name="izz" value="${(m/12.0)*(x**2 + y**2)}"/>
-        <inertial>
-            <mass value="${m}" />
-            <origin xyz="${o_xyz}" rpy="${o_rpy}" />
-            <inertia
-                 ixx="${ixx}" ixy="0.0" ixz="0.0"
-                 iyy="${iyy}" iyz="0.0"
-                 izz="${izz}" />
-        </inertial>
-    </xacro:macro>
-    <xacro:macro name="cylinder_inertia" params="m r l o_xyz o_rpy">
-        <inertial>
-            <mass value="${m}" />
-            <origin xyz="${o_xyz}" rpy="${o_rpy}" />
-            <inertia ixx="${(m/12) * (3*r*r + l*l)}" ixy="0" ixz="0"
-                    iyy="${(m/12) * (3*r*r + l*l)}" iyz="0"
-                    izz="${(m/2) * (r*r)}" />
-        </inertial>
-    </xacro:macro>
-    <xacro:macro name="sphere_inertia" params="m r o_xyz o_rpy">
-        <inertial>
-            <mass value="${m}" />
-            <origin xyz="${o_xyz}" rpy="${o_rpy}" />
-            <inertia ixx="${(2/5) * m * r * r}" ixy="0" ixz="0"
-                    iyy="${(2/5) * m * r * r}" iyz="0"
-                    izz="${(2/5) * m * r * r}" />
-        </inertial>
-    </xacro:macro>
-</robot>
+/home/rakesh/ros2_ws/src/differential_drive/dd_robot/urdf/common_properties.xacro

File: install/dd_robot/share/dd_robot/urdf/mobile_base.xacro (robot description, xacro)
@@ -1,206 +1 @@
-<?xml version="1.0"?>
-<robot xmlns:xacro="http://www.ros.org/wiki/xacro">
-    <xacro:property name="base_length" value="0.6" />
-    <xacro:property name="base_width" value="0.4" />
-    <xacro:property name="base_height" value="0.2" />
-    <xacro:property name="wheel_radius" value="0.1" />
-    <xacro:property name="wheel_length" value="0.05" />
-    <xacro:property name="com_z" value="${base_height/2.0}"/>
-    <link name ="base_footprint" />
-    <link name="base_link">
-        <visual>
-            <geometry>
-                <box size="0.6 0.4 0.2" />
-            </geometry>
-            <origin xyz="0 0 0.1" rpy="0 0 0" />
-            <material name="green" />
-        </visual>
-        <collision>
-            <origin xyz="0 0 0.1" rpy="0 0 0" />
-            <geometry>
-                <box size="0.6 0.4 0.2" />
-            </geometry>
-        </collision>
-        <xacro:box_inertia m="5.0" x="0.6" y="0.4" z="0.2" o_xyz="0 0 0.1" o_rpy="0 0 0" />
-    </link>
-    <link name="right_wheel_link">
-            <visual>
-                <geometry>
-                    <cylinder radius="0.1" length="0.05" />
-                </geometry>
-                <origin xyz="0 0 0" rpy="${pi / 2.0} 0 0" />
-                <material name="gray" />
-            </visual>
-            <collision>
-                <origin xyz="0 0 0" rpy="${pi / 2.0} 0 0" />
-                <geometry>
-                    <cylinder radius="0.1" length="0.05" />
-                </geometry>
-            </collision>
-            <xacro:cylinder_inertia m="1.0" r="0.1" l="0.05"  o_xyz="0 0 0" o_rpy="${pi / 2.0} 0 0" />
-    </link>
-    <link name="left_wheel_link">
-            <visual>
-                <geometry>
-                    <cylinder radius="0.1" length="0.05" />
-                </geometry>
-                <origin xyz="0 0 0" rpy="${pi / 2.0} 0 0" />
-                <material name="gray" />
-            </visual>
-            <collision>
-                <origin xyz="0 0 0" rpy="${pi / 2.0} 0 0" />
-                <geometry>
-                    <cylinder radius="0.1" length="0.05" />
-                </geometry>
-            </collision>
-            <xacro:cylinder_inertia m="1.0" r="0.1" l="0.05" o_xyz="0 0 0" o_rpy="${pi / 2.0} 0 0" />
-    </link>
-    <link name="caster_wheel_link">
-        <visual>
-            <geometry>
-                <sphere radius="0.05" />
-            </geometry>
-            <origin xyz="0 0 0" rpy="0 0 0" />
-            <material name="gray" />
-        </visual>
-        <collision>
-            <origin xyz="0 0 0" rpy="0 0 0" />
-            <geometry>
-                <sphere radius="0.05" />
-            </geometry>
-        </collision>
-        <xacro:sphere_inertia m="0.5" r="0.05" o_xyz="0 0 0" o_rpy="0 0 0" />
-    </link>
-    <!--LIDAR LINK-->
-    <link name="lidar_link">
-        <visual>
-            <geometry>
-                <cylinder radius="0.1" length="0.05" />
-            </geometry>
-            <origin xyz="0 0 0" rpy="${pi} 0 0" />
-            <material name="gray" />
-        </visual>
-        <collision>
-            <origin xyz="0 0 0" rpy="${pi} 0 0" />
-            <geometry>
-                <cylinder radius="0.1" length="0.05" />
-            </geometry>
-        </collision>
-        <xacro:cylinder_inertia m="1.0" r="0.1" l="0.1" o_xyz="0 0 0" o_rpy="${pi} 0 0" />
-    </link>
-    <!--IMU LINK-->
-    <link name="imu_link">
-      <visual>
-         <geometry>
-            <box size="0.1 0.1 0.1"/>
-         </geometry>
-         <origin xyz="0 0 0" rpy="0 0 0"/>
-         <material name="gray"/>
-      </visual>
-      <collision>
-          <origin xyz="0 0 0" rpy="0 0 0"/>
-          <geometry>
-             <box size="0.1 0.1 0.1"/>
-          </geometry>
-      </collision>
-      <inertial>
-         <mass value="0.1"/>
-         <origin xyz="0 0 0" rpy="0 0 0"/>
-         <inertia ixx="0.00033" iyy="0.00033" izz="0.00033" ixy="0" ixz="0" iyz="0"/>
-      </inertial>
-    </link>
-    <joint name="imu_joint" type="fixed">
-       <parent link="base_link"/>
-       <child link="imu_link"/>
-       <origin xyz="0 0 0.1" rpy="0 0 0"/>
-    </joint>
-    <!--CAMERA LINK-->
-    <link name="camera_link">
-         <visual>
-            <origin xyz="0 0 0" rpy="0 0 0"/>
-            <geometry>
-                <box size="0.015 0.130 0.022"/>
-            </geometry>
-         </visual>
-         <collision>
-            <origin xyz="0 0 0" rpy="0 0 0"/>
-            <geometry>
-                <box size="0.015 0.130 0.022"/>
-            </geometry>
-         </collision>
-         <inertial>
-            <origin xyz="0 0 0" rpy="0 0 0"/>
-            <mass value="0.035"/>
-            <inertia ixx="0.001"  ixy="0"  ixz="0" iyy="0.001" iyz="0" izz="0.001" />
-         </inertial>
-    </link>
-    <joint name="camera_joint" type="fixed">
-        <parent link="base_link"/>
-        <child link="camera_link"/>
-        <origin xyz="0.3 0 0.1" rpy="0 0 0"/>
-    </joint>
-    <link name="camera_depth_frame"/>
-    <joint name="camera_depth_joint" type="fixed">
-         <origin xyz="0 0 0" rpy="${-pi/2} 0 ${-pi/2}"/>
-         <parent link="camera_link"/>
-         <child link="camera_depth_frame"/>
-    </joint>
-    <joint name = "base_joint" type ="fixed">
-        <parent link="base_footprint" />
-        <child link = "base_link" />
-        <origin xyz = "0 0 0.1" rpy ="0 0 0" />
-    </joint>
-    <joint name="right_wheel_joint" type="continuous">
-        <parent link="base_link" />
-        <child link="right_wheel_link" />
-        <origin xyz="-0.15 -0.225 0" rpy="0 0 0" />
-        <axis xyz="0 1 0" />
-        <limit effort ="50000" velocity ="10" />
-        <dynamics damping ="1.0" friction="1.0"/>
-    </joint>
-    <joint name="left_wheel_joint" type="continuous">
-        <parent link="base_link" />
-        <child link="left_wheel_link" />
-        <origin xyz="-0.15 0.225 0" rpy="0 0 0" />
-        <axis xyz="0 1 0" />
-        <limit effort ="50000" velocity ="10" />
-        <dynamics damping ="1.0" friction="1.0"/>
-    </joint>
-    <joint name="base_lidar_joint" type="fixed">
-        <parent link="base_link" />
-        <child link="lidar_link" />
-        <origin xyz="0.15 0 0.225" rpy="0 0 0" />
-        <axis xyz="0 1 0" />
-    </joint>
-    <joint name="base_caster_wheel_joint" type="fixed">
-        <parent link="base_link" />
-        <child link="caster_wheel_link" />
-        <origin xyz="0.2 0 -0.05" rpy="0 0 0" />
-    </joint>
-    <!--ros2_control name="GazeboSimSystem" type="system">
-        <hardware>
-            <plugin>gz_ros2_control/GazeboSimSystem</plugin>
-        </hardware>
-        <joint name="left_wheel_joint">
-            <command_interface name="velocity">
-                <param name="min">-1</param>
-                <param name="max">1</param>
-            </command_interface>
-            <state_interface name="position"/>
-            <state_interface name="velocity"/>
-        </joint>
-        <joint name="right_wheel_joint">
-            <command_interface name="velocity">
-                <param name="min">-1</param>
-                <param name="max">1</param>
-            </command_interface>
-            <state_interface name="position"/>
-            <state_interface name="velocity"/>
-        </joint>
-    </ros2_control>
-    <gazebo>
-        <plugin filename= "gz_ros2_control-system" name="gz_ros2_control::GazeboSimROS2ControlPlugin">
-            <parameters>$(find dd_robot)/config/dd_control.yaml</parameters>
-        </plugin>
-    </gazebo-->
-</robot>
+/home/rakesh/ros2_ws/src/differential_drive/dd_robot/urdf/mobile_base.xacro

File: install/dd_robot/share/dd_robot/urdf/mobile_base_gazebo.xacro (robot description, xacro)
@@ -1,152 +1 @@
-<?xml version="1.0"?>
-<robot name ="dd_robot" xmlns:xacro="http://www.ros.org/wiki/xacro">
-    <physics name="1ms" type="bullet-featherstone">
-      <max_step_size>0.001</max_step_size>
-      <real_time_factor>1.0</real_time_factor>
-    </physics>
-    <!--link name="base_link">
-        <collision>
-            <origin xyz="0 0 0.1" rpy="0 0 0" />
-            <geometry>
-                <box size="0.6 0.4 0.2" />
-            </geometry>
-        </collision>
-        <material>Gazebo/Green</material>
-    </link-->
-    <gazebo reference ="caster_wheel_link">
-        <mu1>0.000002</mu1>
-        <mu2>0.000002</mu2>
-        <kp>10000000.0</kp>
-        <kd>1000.0</kd>
-        <material>Gazebo/Yellow</material>
-    </gazebo>
-    <gazebo reference="left_wheel_link">
-        <material>Gazebo/Yellow</material>
-        <mu1>0.2</mu1>
-        <mu2>0.2</mu2>
-        <kp>10000000.0</kp>
-        <kd>1000.0</kd>
-    </gazebo>
-    <gazebo reference="right_wheel_link">
-        <material>Gazebo/Yellow</material>
-        <mu1>0.2</mu1>
-        <mu2>0.2</mu2>
-        <kp>10000000.0</kp>
-        <kd>1000.0</kd>
-    </gazebo>
-    <gazebo reference="lidar_link">
-        <material>Gazebo/Black</material>
-    </gazebo>
-    <gazebo reference ="base_link">
-      <material>Gazebo/Green</material>
-    </gazebo>
-    <gazebo>
-        <plugin
-            filename="gz-sim-diff-drive-system" name="gz::sim::systems::DiffDrive">
-            <odom_topic>/odom</odom_topic>
-            <odom_publish_frequency>20.0</odom_publish_frequency>
-            <left_joint>left_wheel_joint</left_joint>
-            <right_joint>right_wheel_joint</right_joint>
-            <wheel_separation>0.45</wheel_separation>
-            <wheel_radius>0.1</wheel_radius>
-            <frame_id>odom</frame_id>
-            <child_frame_id>base_footprint</child_frame_id>
-            <publish_tf>false</publish_tf>   <!--EKF is already active and publish odom-->
-        </plugin>
-    </gazebo>
-    <gazebo>
-        <plugin
-            filename="gz-sim-joint-state-publisher-system" name="gz::sim::systems::JointStatePublisher">
-            <joint_name>right_wheel_joint</joint_name>
-            <joint_name>left_wheel_joint</joint_name>
-        </plugin>
-    </gazebo>
-    <gazebo>
-      <plugin filename="gz-sim-sensors-system" name="gz::sim::systems::Sensors">
-        <render_engine>ogre2</render_engine>
-      </plugin>
-    </gazebo>
-    <!--LIDAR SENSOR-->
-    <gazebo reference="lidar_link">
-        <sensor name="lidar" type="gpu_lidar">
-           <always_on>1</always_on>
-           <topic>lidar_points</topic>
-           <visualize>true</visualize>
-           <gz_frame_id>lidar_link</gz_frame_id>
-           <update_rate>10.0</update_rate>
-           <lidar>
-               <scan>
-                 <horizontal>
-                   <samples>480</samples>
-                   <resolution>1</resolution>
-                   <min_angle>-3.14159265</min_angle>
-                   <max_angle>3.14159265</max_angle>
-                 </horizontal>
-               </scan>
-               <range>
-                 <min>0.5</min>
-                 <max>131.0</max>
-                 <resolution>0.001</resolution>
-               </range>
-               <noise>
-                 <type>gaussian</type>
-                 <mean>0.0</mean>
-                 <stddev>0.08</stddev>
-               </noise>
-               <frame_id>lidar_link</frame_id>
-           </lidar>
-        </sensor>
-    </gazebo>
-    <gazebo reference="imu_link">
-           <sensor type="imu" name="imu_sensor">
-           <topic>/imu</topic>
-           <gz_frame_id>imu_link</gz_frame_id>
-           <always_on>1</always_on>
-           <update_rate>250</update_rate>
-           <visualize>true</visualize>
-           <imu>
-              <angular_velocity>
-                 <x><noise type="gaussian"><mean>0.0</mean><stddev>0.0002</stddev></noise></x>
-                 <y><noise type="gaussian"><mean>0.0</mean><stddev>0.0002</stddev></noise></y>
-                 <z><noise type="gaussian"><mean>0.0</mean><stddev>0.0002</stddev></noise></z>
-              </angular_velocity>
-              <linear_acceleration>
-                  <x><noise type="gaussian"><mean>0.0</mean><stddev>0.017</stddev></noise></x>
-                  <y><noise type="gaussian"><mean>0.0</mean><stddev>0.017</stddev></noise></y>
-                  <z><noise type="gaussian"><mean>0.0</mean><stddev>0.017</stddev></noise></z>
-              </linear_acceleration>
-           </imu>
-              <plugin filename="gz-sim-imu-system" name="gz::sim::systems::Imu">
-                <initial_orientation_as_reference>false</initial_orientation_as_reference>
-              </plugin>
-          </sensor>
-   </gazebo>
-    <gazebo reference="camera_link">
-      <sensor name="depth_camera" type="rgbd_camera">
-         <always_on>true</always_on>
-         <visualize>true</visualize>
-         <update_rate>20</update_rate>
-         <topic>depth_camera</topic>
-         <gz_frame_id>camera_link</gz_frame_id>
-         <camera>
-          <horizontal_fov>1.047198</horizontal_fov>
-          <image>
-              <width>640</width>
-              <height>480</height>
-              <format>R8G8B8</format>
-          </image>
-          <clip>
-            <near>0.05</near>
-            <far>3</far>
-          </clip>
-          </camera>
-            <!--ros>
-              <remapping>~/image:=/camera/color/image_raw</remapping>
-              <remapping>~/camera_info:=/camera/color/camera_info</remapping>
-              <remapping>~/depth_image:=/camera/depth/image_raw</remapping>
-              <remapping>~/points:=/camera/depth/points</remapping>
-            </ros>
-            <output_type>sensor_msgs/Image</output_type-->
-        </sensor>
-    </gazebo>
-</robot>
+/home/rakesh/ros2_ws/src/differential_drive/dd_robot/urdf/mobile_base_gazebo.xacro

File: install/dd_robot/share/dd_robot/urdf/robot.urdf.xacro (robot description, xacro)
@@ -1,8 +1 @@
-<?xml version="1.0"?>
-<robot name="dd_robot" xmlns:xacro="http://www.ros.org/wiki/xacro">
-    <xacro:include filename="$(find dd_robot)/urdf/common_properties.xacro" />
-    <xacro:include filename="$(find dd_robot)/urdf/mobile_base.xacro" />
-    <xacro:include filename="$(find dd_robot)/urdf/mobile_base_gazebo.xacro" />
- <!--   <xacro:include filename="$(find dd_robot)/urdf/robot_control.xacro" />  -->
-<!--  <xacro:include filename="$(find dd_robot)/urdf/transmission.xacro" />  -->
-</robot>
+/home/rakesh/ros2_ws/src/differential_drive/dd_robot/urdf/robot.urdf.xacro

File: install/dd_robot/share/dd_robot/urdf/robot_control.xacro (robot description, xacro)
@@ -1,26 +1 @@
-<?xml version="1.0"?>
-<robot xmlns:xacro="http://www.ros.org/wiki/xacro">
-    <ros2_control name="dd_robot_ros2_control" type="system">
-        <hardware>
-            <plugin>gz_ros2_control/GazeboSimSystem</plugin>
-        </hardware>
-        <joint name="left_wheel_joint">
-            <command_interface name="velocity"/>
-            <state_interface name="position"/>
-            <state_interface name="velocity"/>
-        </joint>
-        <joint name="right_wheel_joint">
-            <command_interface name="velocity"/>
-            <state_interface name="position"/>
-            <state_interface name="velocity"/>
-        </joint>
-    </ros2_control>
-    <gazebo>
-        <plugin name="gz_ros2_control::GazeboSimROS2ControlPlugin" filename="gz_ros2_control-system">
-            <robot_param>robot_description</robot_param>
-            <parameters>$(find dd_robot)/config/dd_control.yaml</parameters>
-            <plugin filename="gz-sim-imu-system" name="gz::sim::systems::Imu">
-            </plugin>
-        </plugin>
-    </gazebo>
-</robot>
+/home/rakesh/ros2_ws/src/differential_drive/dd_robot/urdf/robot_control.xacro

File: install/dd_robot/share/dd_robot/urdf/transmission.xacro (robot description, xacro)
@@ -1,21 +1 @@
-<?xml version="1.0"?>
-<robot xmlns:xacro="http://www.ros.org/wiki/xacro">
-    <transmission name="left_wheel_trans">
-        <type>transmission_interface/SimpleTransmission</type>
-        <joint name="left_wheel_joint">
-            <hardwareInterface>hardware_interface/VelocityJointInterface</hardwareInterface>  <!-- Or PositionJointInterface for hardware -->
-        </joint>
-        <actuator name="left_wheel_motor">
-            <mechanical_reduction>1</mechanical_reduction>  <!-- Gear ratio; 1 for direct drive -->
-        </actuator>
-    </transmission>
-    <transmission name="right_wheel_trans">
-        <type>transmission_interface/SimpleTransmission</type>
-        <joint name="right_wheel_joint">
-            <hardwareInterface>hardware_interface/VelocityJointInterface</hardwareInterface>
-        </joint>
-        <actuator name="right_wheel_motor">
-            <mechanical_reduction>1</mechanical_reduction>
-        </actuator>
-    </transmission>
-</robot>
+/home/rakesh/ros2_ws/src/differential_drive/dd_robot/urdf/transmission.xacro
